Commit message: Add scaling functionality to the rename script

File: gundam_rx78_description/urdf/GGC_TestModel_rx78_20170112_.urdf (robot description, URDF)
Before this commit: robot GGC_TestModel_rx78_20170112, 98 links, 97 joints
Links:
- link head_neck_p_link: mass 1114.42019778 -> 1.1144201977800003; geometry collision mesh filename=package://gundam_rx78_description/meshes/rx78_object_011-li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 scale=0.1 0.1 0.1; visual mesh filename=package://gundam_rx78_description/meshes/rx78_object_011-li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 scale=0.1 0.1 0.1
- link head_neck_y_link: mass 178.861139647 -> 0.17886113964700004; geometry collision mesh filename=package://gundam_rx78_description/meshes/rx78_object_008-li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 scale=0.1 0.1 0.1; visual mesh filename=package://gundam_rx78_description/meshes/rx78_object_008-li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 scale=0.1 0.1 0.1
- link larm_elbow_p2_link: mass 713.563452473 -> 0.7135634524730001; geometry collision mesh filename=package://gundam_rx78_description/meshes/rx78_object_064-li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 scale=0.1 0.1 0.1; visual mesh filename=package://gundam_rx78_description/meshes/rx78_object_064-li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 scale=0.1 0.1 0.1
- link larm_elbow_p_link: mass 299.837062729 -> 0.29983706272900007; geometry collision mesh filename=package://gundam_rx78_description/meshes/rx78_object_062-li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 scale=0.1 0.1 0.1; visual mesh filename=package://gundam_rx78_description/meshes/rx78_object_062-li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 scale=0.1 0.1 0.1
- link larm_gripper_index0_mimic_link: mass 50 -> 0.05000000000000001; geometry collision mesh filename=package://gundam_rx78_description/meshes/rx78_object_056-li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 scale=0.1 0.1 0.1; visual mesh filename=package://gundam_rx78_description/meshes/rx78_object_056-li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 scale=0.1 0.1 0.1
- link larm_gripper_index1_mimic_link: mass 50 -> 0.05000000000000001; geometry collision mesh filename=package://gundam_rx78_description/meshes/rx78_object_055-li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 scale=0.1 0.1 0.1; visual mesh filename=package://gundam_rx78_description/meshes/rx78_object_055-li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 scale=0.1 0.1 0.1
- link larm_gripper_index2_mimic_link: mass 50 -> 0.05000000000000001; geometry collision mesh filename=package://gundam_rx78_description/meshes/rx78_object_054-li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 scale=0.1 0.1 0.1; visual mesh filename=package://gundam_rx78_description/meshes/rx78_object_054-li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 scale=0.1 0.1 0.1
- link larm_gripper_link: mass 50 -> 0.05000000000000001; geometry collision mesh filename=package://gundam_rx78_description/meshes/rx78_object_059-li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 scale=0.1 0.1 0.1; visual mesh filename=package://gundam_rx78_description/meshes/rx78_object_059-li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 scale=0.1 0.1 0.1
- link larm_gripper_little0_mimic_link: mass 50 -> 0.05000000000000001; geometry collision mesh filename=package://gundam_rx78_description/meshes/rx78_object_053-li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 scale=0.1 0.1 0.1; visual mesh filename=package://gundam_rx78_description/meshes/rx78_object_053-li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 scale=0.1 0.1 0.1
- link larm_gripper_little1_mimic_link: mass 50 -> 0.05000000000000001; geometry collision mesh filename=package://gundam_rx78_description/meshes/rx78_object_052-li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 scale=0.1 0.1 0.1; visual mesh filename=package://gundam_rx78_description/meshes/rx78_object_052-li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 scale=0.1 0.1 0.1
- link larm_gripper_little2_mimic_link: mass 50 -> 0.05000000000000001; geometry collision mesh filename=package://gundam_rx78_description/meshes/rx78_object_071-li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 scale=0.1 0.1 0.1; visual mesh filename=package://gundam_rx78_description/meshes/rx78_object_071-li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 scale=0.1 0.1 0.1
- link larm_gripper_middle0_mimic_link: mass 50 -> 0.05000000000000001; geometry collision mesh filename=package://gundam_rx78_description/meshes/rx78_object_067-li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 scale=0.1 0.1 0.1; visual mesh filename=package://gundam_rx78_description/meshes/rx78_object_067-li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 scale=0.1 0.1 0.1
- link larm_gripper_middle1_mimic_link: mass 50 -> 0.05000000000000001; geometry collision mesh filename=package://gundam_rx78_description/meshes/rx78_object_066-li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 scale=0.1 0.1 0.1; visual mesh filename=package://gundam_rx78_description/meshes/rx78_object_066-li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 scale=0.1 0.1 0.1
- link larm_gripper_middle2_mimic_link: mass 50 -> 0.05000000000000001; geometry collision mesh filename=package://gundam_rx78_description/meshes/rx78_object_065-li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 scale=0.1 0.1 0.1; visual mesh filename=package://gundam_rx78_description/meshes/rx78_object_065-li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 scale=0.1 0.1 0.1
- link larm_gripper_ring0_mimic_link: mass 50 -> 0.05000000000000001; geometry collision mesh filename=package://gundam_rx78_description/meshes/rx78_object_070-li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 scale=0.1 0.1 0.1; visual mesh filename=package://gundam_rx78_description/meshes/rx78_object_070-li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 scale=0.1 0.1 0.1
- link larm_gripper_ring1_mimic_link: mass 50 -> 0.05000000000000001; geometry collision mesh filename=package://gundam_rx78_description/meshes/rx78_object_069-li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 scale=0.1 0.1 0.1; visual mesh filename=package://gundam_rx78_description/meshes/rx78_object_069-li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 scale=0.1 0.1 0.1
- link larm_gripper_ring2_mimic_link: mass 50 -> 0.05000000000000001; geometry collision mesh filename=package://gundam_rx78_description/meshes/rx78_object_068-li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 scale=0.1 0.1 0.1; visual mesh filename=package://gundam_rx78_description/meshes/rx78_object_068-li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 scale=0.1 0.1 0.1
- link larm_gripper_thumb1_mimic_link: mass 50 -> 0.05000000000000001; geometry collision mesh filename=package://gundam_rx78_description/meshes/rx78_object_058-li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 scale=0.1 0.1 0.1; visual mesh filename=package://gundam_rx78_description/meshes/rx78_object_058-li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 scale=0.1 0.1 0.1
- link larm_gripper_thumb2_mimic_link: mass 50 -> 0.05000000000000001; geometry collision mesh filename=package://gundam_rx78_description/meshes/rx78_object_057-li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 scale=0.1 0.1 0.1; visual mesh filename=package://gundam_rx78_description/meshes/rx78_object_057-li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 scale=0.1 0.1 0.1
- link larm_shoulder_p_link: mass 70.6689458051 -> 0.07066894580510001; geometry collision mesh filename=package://gundam_rx78_description/meshes/rx78_object_063-li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 scale=0.1 0.1 0.1; visual mesh filename=package://gundam_rx78_description/meshes/rx78_object_063-li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 scale=0.1 0.1 0.1
- link larm_shoulder_r_link: mass 383.847721533 -> 0.3838477215330001; geometry collision mesh filename=package://gundam_rx78_description/meshes/rx78_object_001-li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 scale=0.1 0.1 0.1; visual mesh filename=package://gundam_rx78_description/meshes/rx78_object_001-li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 scale=0.1 0.1 0.1
- link larm_shoulder_y_link: mass 267.165510727 -> 0.26716551072700007; geometry collision mesh filename=package://gundam_rx78_description/meshes/rx78_object_002-li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 scale=0.1 0.1 0.1; visual mesh filename=package://gundam_rx78_description/meshes/rx78_object_002-li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 scale=0.1 0.1 0.1
- link larm_wrist_r_link: mass 59.0272892404 -> 0.059027289240400016; geometry collision mesh filename=package://gundam_rx78_description/meshes/rx78_object_060-li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 scale=0.1 0.1 0.1; visual mesh filename=package://gundam_rx78_description/meshes/rx78_object_060-li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 scale=0.1 0.1 0.1
- link larm_wrist_y_link: mass 50 -> 0.05000000000000001; geometry collision mesh filename=package://gundam_rx78_description/meshes/rx78_object_061-li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 scale=0.1 0.1 0.1; visual mesh filename=package://gundam_rx78_description/meshes/rx78_object_061-li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 scale=0.1 0.1 0.1
- link lleg_ankle_p_link: mass 390.3954127 -> 0.3903954127000001; geometry collision mesh filename=package://gundam_rx78_description/meshes/rx78_object_040-li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 scale=0.1 0.1 0.1; visual mesh filename=package://gundam_rx78_description/meshes/rx78_object_040-li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 scale=0.1 0.1 0.1
- link lleg_ankle_p_mimic_link: mass 773.357103509 -> 0.7733571035090002; geometry collision mesh filename=package://gundam_rx78_description/meshes/rx78_object_039-li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 scale=0.1 0.1 0.1; visual mesh filename=package://gundam_rx78_description/meshes/rx78_object_039-li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 scale=0.1 0.1 0.1
- link lleg_ankle_r_link: mass 917.386968391 -> 0.9173869683910002; geometry collision mesh filename=package://gundam_rx78_description/meshes/rx78_object_034-li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 scale=0.1 0.1 0.1; visual mesh filename=package://gundam_rx78_description/meshes/rx78_object_034-li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 scale=0.1 0.1 0.1
- link lleg_ankle_r_mimic_link: mass 328.651860737 -> 0.3286518607370001; geometry collision mesh filename=package://gundam_rx78_description/meshes/rx78_object_032-li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 scale=0.1 0.1 0.1; visual mesh filename=package://gundam_rx78_description/meshes/rx78_object_032-li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 scale=0.1 0.1 0.1
- link lleg_crotch_p_back_mimic_link: mass 164.944289475 -> 0.16494428947500003; geometry collision mesh filename=package://gundam_rx78_description/meshes/rx78_object_027-li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 scale=0.1 0.1 0.1; visual mesh filename=package://gundam_rx78_description/meshes/rx78_object_027-li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 scale=0.1 0.1 0.1
- link lleg_crotch_p_front_mimic_link: mass 164.944271247 -> 0.16494427124700003; geometry collision mesh filename=package://gundam_rx78_description/meshes/rx78_object_028-li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 scale=0.1 0.1 0.1; visual mesh filename=package://gundam_rx78_description/meshes/rx78_object_028-li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 scale=0.1 0.1 0.1
- link lleg_crotch_p_link: mass 204.8 -> 0.20480000000000007
- link lleg_crotch_r_link: mass 282.636837959 -> 0.2826368379590001; geometry collision mesh filename=package://gundam_rx78_description/meshes/rx78_object_029-li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 scale=0.1 0.1 0.1; visual mesh filename=package://gundam_rx78_description/meshes/rx78_object_029-li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 scale=0.1 0.1 0.1
- link lleg_crotch_r_mimic_link: mass 225.268736797 -> 0.22526873679700005; geometry collision mesh filename=package://gundam_rx78_description/meshes/rx78_object_043-li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 scale=0.1 0.1 0.1; visual mesh filename=package://gundam_rx78_description/meshes/rx78_object_043-li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 scale=0.1 0.1 0.1
- link lleg_crotch_y_link: mass 1373.45774708 -> 1.3734577470800002; geometry collision mesh filename=package://gundam_rx78_description/meshes/rx78_object_042-li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 scale=0.1 0.1 0.1; visual mesh filename=package://gundam_rx78_description/meshes/rx78_object_042-li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 scale=0.1 0.1 0.1
- link lleg_knee_p2_link: mass 5927.78010448 -> 5.927780104480001; geometry collision mesh filename=package://gundam_rx78_description/meshes/rx78_object_030-li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 scale=0.1 0.1 0.1; visual mesh filename=package://gundam_rx78_description/meshes/rx78_object_030-li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 scale=0.1 0.1 0.1
- link lleg_knee_p_link: mass 536.138633274 -> 0.5361386332740001; geometry collision mesh filename=package://gundam_rx78_description/meshes/rx78_object_041-li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 scale=0.1 0.1 0.1; visual mesh filename=package://gundam_rx78_description/meshes/rx78_object_041-li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 scale=0.1 0.1 0.1
- link rarm_elbow_p2_link: mass 706.005068182 -> 0.7060050681820002; geometry collision mesh filename=package://gundam_rx78_description/meshes/rx78_object_075-li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 scale=0.1 0.1 0.1; visual mesh filename=package://gundam_rx78_description/meshes/rx78_object_075-li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 scale=0.1 0.1 0.1
- link rarm_elbow_p_link: mass 283.033251041 -> 0.2830332510410001; geometry collision mesh filename=package://gundam_rx78_description/meshes/rx78_object_076-li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 scale=0.1 0.1 0.1; visual mesh filename=package://gundam_rx78_description/meshes/rx78_object_076-li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 scale=0.1 0.1 0.1
- link rarm_gripper_index0_mimic_link: mass 50 -> 0.05000000000000001; geometry collision mesh filename=package://gundam_rx78_description/meshes/rx78_object_017-li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 scale=0.1 0.1 0.1; visual mesh filename=package://gundam_rx78_description/meshes/rx78_object_017-li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 scale=0.1 0.1 0.1
- link rarm_gripper_index1_mimic_link: mass 50 -> 0.05000000000000001; geometry collision mesh filename=package://gundam_rx78_description/meshes/rx78_object_016-li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 scale=0.1 0.1 0.1; visual mesh filename=package://gundam_rx78_description/meshes/rx78_object_016-li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 scale=0.1 0.1 0.1
- link rarm_gripper_index2_mimic_link: mass 50 -> 0.05000000000000001; geometry collision mesh filename=package://gundam_rx78_description/meshes/rx78_object_015-li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 scale=0.1 0.1 0.1; visual mesh filename=package://gundam_rx78_description/meshes/rx78_object_015-li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 scale=0.1 0.1 0.1
- link rarm_gripper_link: mass 50 -> 0.05000000000000001; geometry collision mesh filename=package://gundam_rx78_description/meshes/rx78_object_051-li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 scale=0.1 0.1 0.1; visual mesh filename=package://gundam_rx78_description/meshes/rx78_object_051-li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 scale=0.1 0.1 0.1
- link rarm_gripper_little0_mimic_link: mass 50 -> 0.05000000000000001; geometry collision mesh filename=package://gundam_rx78_description/meshes/rx78_object_020-li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 scale=0.1 0.1 0.1; visual mesh filename=package://gundam_rx78_description/meshes/rx78_object_020-li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 scale=0.1 0.1 0.1
- link rarm_gripper_little1_mimic_link: mass 50 -> 0.05000000000000001; geometry collision mesh filename=package://gundam_rx78_description/meshes/rx78_object_019-li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 scale=0.1 0.1 0.1; visual mesh filename=package://gundam_rx78_description/meshes/rx78_object_019-li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 scale=0.1 0.1 0.1
- link rarm_gripper_little2_mimic_link: mass 50 -> 0.05000000000000001; geometry collision mesh filename=package://gundam_rx78_description/meshes/rx78_object_018-li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 scale=0.1 0.1 0.1; visual mesh filename=package://gundam_rx78_description/meshes/rx78_object_018-li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 scale=0.1 0.1 0.1
- link rarm_gripper_middle0_mimic_link: mass 50 -> 0.05000000000000001; geometry collision mesh filename=package://gundam_rx78_description/meshes/rx78_object_014-li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 scale=0.1 0.1 0.1; visual mesh filename=package://gundam_rx78_description/meshes/rx78_object_014-li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 scale=0.1 0.1 0.1
- link rarm_gripper_middle1_mimic_link: mass 50 -> 0.05000000000000001; geometry collision mesh filename=package://gundam_rx78_description/meshes/rx78_object_013-li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 scale=0.1 0.1 0.1; visual mesh filename=package://gundam_rx78_description/meshes/rx78_object_013-li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 scale=0.1 0.1 0.1
- link rarm_gripper_middle2_mimic_link: mass 50 -> 0.05000000000000001; geometry collision mesh filename=package://gundam_rx78_description/meshes/rx78_object_012-li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 scale=0.1 0.1 0.1; visual mesh filename=package://gundam_rx78_description/meshes/rx78_object_012-li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 scale=0.1 0.1 0.1
- link rarm_gripper_ring0_mimic_link: mass 50 -> 0.05000000000000001; geometry collision mesh filename=package://gundam_rx78_description/meshes/rx78_object_074-li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 scale=0.1 0.1 0.1; visual mesh filename=package://gundam_rx78_description/meshes/rx78_object_074-li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 scale=0.1 0.1 0.1
- link rarm_gripper_ring1_mimic_link: mass 50 -> 0.05000000000000001; geometry collision mesh filename=package://gundam_rx78_description/meshes/rx78_object_073-li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 scale=0.1 0.1 0.1; visual mesh filename=package://gundam_rx78_description/meshes/rx78_object_073-li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 scale=0.1 0.1 0.1
- link rarm_gripper_ring2_mimic_link: mass 50 -> 0.05000000000000001; geometry collision mesh filename=package://gundam_rx78_description/meshes/rx78_object_072-li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 scale=0.1 0.1 0.1; visual mesh filename=package://gundam_rx78_description/meshes/rx78_object_072-li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 scale=0.1 0.1 0.1
- link rarm_gripper_thumb1_mimic_link: mass 50 -> 0.05000000000000001; geometry collision mesh filename=package://gundam_rx78_description/meshes/rx78_object_050-li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 scale=0.1 0.1 0.1; visual mesh filename=package://gundam_rx78_description/meshes/rx78_object_050-li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 scale=0.1 0.1 0.1
- link rarm_gripper_thumb2_mimic_link: mass 50 -> 0.05000000000000001; geometry collision mesh filename=package://gundam_rx78_description/meshes/rx78_object_049-li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 scale=0.1 0.1 0.1; visual mesh filename=package://gundam_rx78_description/meshes/rx78_object_049-li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 scale=0.1 0.1 0.1
- link rarm_shoulder_p_link: mass 70.6689430644 -> 0.07066894306440001; geometry collision mesh filename=package://gundam_rx78_description/meshes/rx78_object_078-li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 scale=0.1 0.1 0.1; visual mesh filename=package://gundam_rx78_description/meshes/rx78_object_078-li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 scale=0.1 0.1 0.1
- link rarm_shoulder_r_link: mass 368.19225087 -> 0.36819225087000007; geometry collision mesh filename=package://gundam_rx78_description/meshes/rx78_object_046-li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 scale=0.1 0.1 0.1; visual mesh filename=package://gundam_rx78_description/meshes/rx78_object_046-li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 scale=0.1 0.1 0.1
- link rarm_shoulder_y_link: mass 263.772287035 -> 0.26377228703500005; geometry collision mesh filename=package://gundam_rx78_description/meshes/rx78_object_077-li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 scale=0.1 0.1 0.1; visual mesh filename=package://gundam_rx78_description/meshes/rx78_object_077-li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 scale=0.1 0.1 0.1
- link rarm_wrist_r_link: mass 59.0272726608 -> 0.05902727266080002; geometry collision mesh filename=package://gundam_rx78_description/meshes/rx78_object_048-li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 scale=0.1 0.1 0.1; visual mesh filename=package://gundam_rx78_description/meshes/rx78_object_048-li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 scale=0.1 0.1 0.1
- link rarm_wrist_y_link: mass 50 -> 0.05000000000000001; geometry collision mesh filename=package://gundam_rx78_description/meshes/rx78_object_047-li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 scale=0.1 0.1 0.1; visual mesh filename=package://gundam_rx78_description/meshes/rx78_object_047-li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 scale=0.1 0.1 0.1
- link rleg_ankle_p_link: mass 780.790853975 -> 0.7807908539750001; geometry collision mesh filename=package://gundam_rx78_description/meshes/rx78_object_022-li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 scale=0.1 0.1 0.1; visual mesh filename=package://gundam_rx78_description/meshes/rx78_object_022-li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 scale=0.1 0.1 0.1
- link rleg_ankle_p_mimic_link: mass 773.399153362 -> 0.7733991533620002; geometry collision mesh filename=package://gundam_rx78_description/meshes/rx78_object_021-li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 scale=0.1 0.1 0.1; visual mesh filename=package://gundam_rx78_description/meshes/rx78_object_021-li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 scale=0.1 0.1 0.1
- link rleg_ankle_r_link: mass 1003.93177287 -> 1.0039317728700003; geometry collision mesh filename=package://gundam_rx78_description/meshes/rx78_object_091-li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 scale=0.1 0.1 0.1; visual mesh filename=package://gundam_rx78_description/meshes/rx78_object_091-li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 scale=0.1 0.1 0.1
- link rleg_ankle_r_mimic_link: mass 312.102482906 -> 0.31210248290600007; geometry collision mesh filename=package://gundam_rx78_description/meshes/rx78_object_089-li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 scale=0.1 0.1 0.1; visual mesh filename=package://gundam_rx78_description/meshes/rx78_object_089-li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 scale=0.1 0.1 0.1
- link rleg_crotch_p_back_mimic_link: mass 164.944262652 -> 0.16494426265200002; geometry collision mesh filename=package://gundam_rx78_description/meshes/rx78_object_025-li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 scale=0.1 0.1 0.1; visual mesh filename=package://gundam_rx78_description/meshes/rx78_object_025-li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 scale=0.1 0.1 0.1
- link rleg_crotch_p_front_mimic_link: mass 164.913885657 -> 0.16491388565700005; geometry collision mesh filename=package://gundam_rx78_description/meshes/rx78_object_085-li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 scale=0.1 0.1 0.1; visual mesh filename=package://gundam_rx78_description/meshes/rx78_object_085-li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 scale=0.1 0.1 0.1
- link rleg_crotch_p_link: mass 204.8 -> 0.20480000000000007
- link rleg_crotch_r_link: mass 282.64330076 -> 0.28264330076000005; geometry collision mesh filename=package://gundam_rx78_description/meshes/rx78_object_086-li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 scale=0.1 0.1 0.1; visual mesh filename=package://gundam_rx78_description/meshes/rx78_object_086-li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 scale=0.1 0.1 0.1
- link rleg_crotch_r_mimic_link: mass 225.268727751 -> 0.22526872775100004; geometry collision mesh filename=package://gundam_rx78_description/meshes/rx78_object_026-li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 scale=0.1 0.1 0.1; visual mesh filename=package://gundam_rx78_description/meshes/rx78_object_026-li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 scale=0.1 0.1 0.1
- link rleg_crotch_y_link: mass 1401.5034554 -> 1.4015034554000003; geometry collision mesh filename=package://gundam_rx78_description/meshes/rx78_object_024-li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 scale=0.1 0.1 0.1; visual mesh filename=package://gundam_rx78_description/meshes/rx78_object_024-li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 scale=0.1 0.1 0.1
- link rleg_knee_p2_link: mass 5351.78567125 -> 5.351785671250001; geometry collision mesh filename=package://gundam_rx78_description/meshes/rx78_object_087-li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 scale=0.1 0.1 0.1; visual mesh filename=package://gundam_rx78_description/meshes/rx78_object_087-li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 scale=0.1 0.1 0.1
- link rleg_knee_p_link: mass 460.391964732 -> 0.4603919647320001; geometry collision mesh filename=package://gundam_rx78_description/meshes/rx78_object_023-li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 scale=0.1 0.1 0.1; visual mesh filename=package://gundam_rx78_description/meshes/rx78_object_023-li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 scale=0.1 0.1 0.1
- link rx78_Null_008_link: mass 50.4267115666 -> 0.05042671156660001; geometry collision mesh filename=package://gundam_rx78_description/meshes/rx78_object_006-li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 scale=0.1 0.1 0.1; visual mesh filename=package://gundam_rx78_description/meshes/rx78_object_006-li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 scale=0.1 0.1 0.1
- link rx78_Null_010_link: mass 50.4267735308 -> 0.05042677353080001; geometry collision mesh filename=package://gundam_rx78_description/meshes/rx78_object_007-li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 scale=0.1 0.1 0.1; visual mesh filename=package://gundam_rx78_description/meshes/rx78_object_007-li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 scale=0.1 0.1 0.1
- link rx78_Null_013_link: mass 1512.48489354 -> 1.5124848935400004; geometry collision mesh filename=package://gundam_rx78_description/meshes/rx78_object_003-li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 scale=0.1 0.1 0.1; visual mesh filename=package://gundam_rx78_description/meshes/rx78_object_003-li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 scale=0.1 0.1 0.1
- link rx78_Null_048_link: mass 1018.88896874 -> 1.0188889687400002; geometry collision mesh filename=package://gundam_rx78_description/meshes/rx78_object_045-li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 scale=0.1 0.1 0.1; visual mesh filename=package://gundam_rx78_description/meshes/rx78_object_045-li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 scale=0.1 0.1 0.1
- link rx78_Null_081_link: mass 664.672905439 -> 0.6646729054390002; geometry collision mesh filename=package://gundam_rx78_description/meshes/rx78_object_079-li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 scale=0.1 0.1 0.1; visual mesh filename=package://gundam_rx78_description/meshes/rx78_object_079-li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 scale=0.1 0.1 0.1
- link rx78_Null_083_link: mass 1467.43234048 -> 1.4674323404800003; geometry collision mesh filename=package://gundam_rx78_description/meshes/rx78_object_044-li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 scale=0.1 0.1 0.1; visual mesh filename=package://gundam_rx78_description/meshes/rx78_object_044-li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 scale=0.1 0.1 0.1
- link torso_lthrust_p_link: mass 204.8 -> 0.20480000000000007
- link torso_lthrust_r_link: mass 51.716551588 -> 0.051716551588000016; geometry collision mesh filename=package://gundam_rx78_description/meshes/rx78_object_004-li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 scale=0.1 0.1 0.1; visual mesh filename=package://gundam_rx78_description/meshes/rx78_object_004-li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 scale=0.1 0.1 0.1
- link torso_rthrust_p_link: mass 204.8 -> 0.20480000000000007
- link torso_rthrust_r_link: mass 51.7165514196 -> 0.051716551419600014; geometry collision mesh filename=package://gundam_rx78_description/meshes/rx78_object_005-li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 scale=0.1 0.1 0.1; visual mesh filename=package://gundam_rx78_description/meshes/rx78_object_005-li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 scale=0.1 0.1 0.1
- link torso_waist_p2_link: mass 4926.49409778 -> 4.926494097780001; geometry collision mesh filename=package://gundam_rx78_description/meshes/rx78_object_080-li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 scale=0.1 0.1 0.1; visual mesh filename=package://gundam_rx78_description/meshes/rx78_object_080-li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 scale=0.1 0.1 0.1
- link torso_waist_p_link: mass 1237.62990073 -> 1.2376299007300002; geometry collision mesh filename=package://gundam_rx78_description/meshes/rx78_object_083-li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 scale=0.1 0.1 0.1; visual mesh filename=package://gundam_rx78_description/meshes/rx78_object_083-li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 scale=0.1 0.1 0.1
- link torso_waist_y_link: mass 942.874289258 -> 0.9428742892580002; geometry collision mesh filename=package://gundam_rx78_description/meshes/rx78_object_084-li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 scale=0.1 0.1 0.1; visual mesh filename=package://gundam_rx78_description/meshes/rx78_object_084-li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 scale=0.1 0.1 0.1
Joints:
- joint head_neck_p_joint: origin xyz=0.0 -0.134118 0.928577 rpy=0.0 -0.0 0.0 -> xyz=0.0 -0.0134118 0.0928577 rpy=0.0 -0.0 0.0
- joint head_neck_y_joint: origin xyz=0.0 0.36632 1.42247 rpy=0.0 -0.0 0.0 -> xyz=0.0 0.036632 0.14224699999999998 rpy=0.0 -0.0 0.0
- joint larm_elbow_p_joint: origin xyz=-2e-07 3.09e-05 -1.55024 rpy=0.0 -0.0 0.0 -> xyz=-2e-08 3.09e-06 -0.15502400000000002 rpy=0.0 -0.0 0.0
- joint larm_gripper_index0_mimic_joint: origin xyz=-0.0683779 -0.31073 -0.853204 rpy=-9.99999997475e-07 -0.0 0.0 -> xyz=-0.006837790000000001 -0.031073000000000003 -0.0853204 rpy=-9.99999997475e-07 -0.0 0.0
- joint larm_gripper_index1_mimic_joint: origin xyz=-0.0498724 -9e-07 -0.295346 rpy=0.0 -9.99999997475e-07 0.0 -> xyz=-0.00498724 -9e-08 -0.0295346 rpy=0.0 -9.99999997475e-07 0.0
- joint larm_gripper_index2_mimic_joint: origin xyz=1e-06 0.0 -0.366374 rpy=-7.0000000959e-06 -4.99999987365e-06 0.0 -> xyz=1e-07 0.0 -0.0366374 rpy=-7.0000000959e-06 -4.99999987365e-06 0.0
- joint larm_gripper_joint: origin xyz=-0.265212 -0.284142 -0.0825119 rpy=0.0 1.99999999495e-06 0.0 -> xyz=-0.0265212 -0.0284142 -0.00825119 rpy=0.0 1.99999999495e-06 0.0
- joint larm_gripper_little0_mimic_joint: origin xyz=-0.0683781 -0.105633 -0.877139 rpy=-9.99999997475e-07 -0.0 0.0 -> xyz=-0.00683781 -0.010563300000000001 -0.08771390000000001 rpy=-9.99999997475e-07 -0.0 0.0
- joint larm_gripper_little1_mimic_joint: origin xyz=-0.0498724 -7e-07 -0.295345 rpy=0.0 -0.0 0.0 -> xyz=-0.00498724 -7e-08 -0.029534500000000005 rpy=0.0 -0.0 0.0
- joint larm_gripper_little2_mimic_joint: origin xyz=1e-06 2e-07 -0.366374 rpy=-6.00000021215e-06 -4.99999987365e-06 0.0 -> xyz=1e-07 2e-08 -0.0366374 rpy=-6.00000021215e-06 -4.99999987365e-06 0.0
- joint larm_gripper_middle0_mimic_joint: origin xyz=-0.0683784 0.310822 -0.782966 rpy=-9.99999997475e-07 -0.0 0.0 -> xyz=-0.006837840000000001 0.0310822 -0.07829660000000001 rpy=-9.99999997475e-07 -0.0 0.0
- joint larm_gripper_middle1_mimic_joint: origin xyz=-0.0498726 -8e-07 -0.295345 rpy=0.0 -0.0 0.0 -> xyz=-0.00498726 -8e-08 -0.029534500000000005 rpy=0.0 -0.0 0.0
- joint larm_gripper_middle2_mimic_joint: origin xyz=1e-06 2e-07 -0.366374 rpy=-9.00000031809e-06 -4.99999987365e-06 0.0 -> xyz=1e-07 2e-08 -0.0366374 rpy=-9.00000031809e-06 -4.99999987365e-06 0.0
- joint larm_gripper_ring0_mimic_joint: origin xyz=-0.0683781 0.0989056 -0.842841 rpy=-9.99999997475e-07 -0.0 0.0 -> xyz=-0.00683781 0.00989056 -0.0842841 rpy=-9.99999997475e-07 -0.0 0.0
- joint larm_gripper_ring1_mimic_joint: origin xyz=-0.0498724 -7e-07 -0.295345 rpy=0.0 -0.0 0.0 -> xyz=-0.00498724 -7e-08 -0.029534500000000005 rpy=0.0 -0.0 0.0
- joint larm_gripper_ring2_mimic_joint: origin xyz=1.5e-06 1e-07 -0.366374 rpy=-7.99999997963e-06 -4.99999987365e-06 0.0 -> xyz=1.5000000000000002e-07 1e-08 -0.0366374 rpy=-7.99999997963e-06 -4.99999987365e-06 0.0
- joint larm_gripper_thumb1_mimic_joint: origin xyz=4e-07 -0.248849 -0.170409 rpy=0.0 -0.0 0.0 -> xyz=4e-08 -0.0248849 -0.0170409 rpy=0.0 -0.0 0.0
- joint larm_gripper_thumb2_mimic_joint: origin xyz=1.7e-06 -2.49e-05 -0.366318 rpy=-9.99999997475e-07 -0.0 0.0 -> xyz=1.7000000000000001e-07 -2.49e-06 -0.0366318 rpy=-9.99999997475e-07 -0.0 0.0
- joint larm_shoulder_p_joint: origin xyz=1.72 0.369688 1.07247 rpy=0.0 -0.0 0.0 -> xyz=0.17200000000000001 0.0369688 0.10724700000000001 rpy=0.0 -0.0 0.0
- joint larm_shoulder_r_joint: origin xyz=0.93 -0.0191881 0.0 rpy=0.0 -0.0 0.0 -> xyz=0.09300000000000001 -0.00191881 0.0 rpy=0.0 -0.0 0.0
- joint larm_shoulder_y_joint: origin xyz=4e-07 0.0 -0.604907 rpy=0.0 -0.0 0.0 -> xyz=4e-08 0.0 -0.0604907 rpy=0.0 -0.0 0.0
- joint larm_wrist_r_joint: origin xyz=0.136895 -1e-07 -0.239744 rpy=9.99999997475e-07 -0.0 0.0 -> xyz=0.0136895 -1e-08 -0.023974400000000003 rpy=9.99999997475e-07 -0.0 0.0
- joint larm_wrist_y_joint: origin xyz=-8e-07 -3.07e-05 -2.51486 rpy=0.0 9.99999997475e-07 0.0 -> xyz=-8e-08 -3.0700000000000003e-06 -0.25148600000000004 rpy=0.0 9.99999997475e-07 0.0
- joint lleg_ankle_p_joint: origin xyz=2.8e-06 0.221803 -6.02553 rpy=0.0 1.99999999495e-06 0.0 -> xyz=2.8e-07 0.0221803 -0.602553 rpy=0.0 1.99999999495e-06 0.0
- joint lleg_ankle_p_mimic_joint: origin xyz=1e-07 -1e-07 0.0 rpy=0.0 -9.99999997475e-07 0.0 -> xyz=1e-08 -1e-08 0.0 rpy=0.0 -9.99999997475e-07 0.0
- joint lleg_ankle_r_joint: origin xyz=2.5e-06 -1.44559 -0.716288 rpy=0.0 -0.0 1.57079632679 -> xyz=2.5000000000000004e-07 -0.144559 -0.0716288 rpy=0.0 -0.0 1.57079632679
- joint lleg_ankle_r_mimic_joint: origin xyz=1.9e-06 -6e-07 -0.716289 rpy=0.0 -0.0 1.57079632679 -> xyz=1.9e-07 -6e-08 -0.0716289 rpy=0.0 -0.0 1.57079632679
- joint lleg_crotch_p_back_mimic_joint: origin xyz=0.76 1.10287 0.470002 rpy=0.0 -0.0 0.0 -> xyz=0.07600000000000001 0.11028700000000001 0.0470002 rpy=0.0 -0.0 0.0
- joint lleg_crotch_p_front_mimic_joint: origin xyz=0.76 -1.09713 0.470002 rpy=0.0 -0.0 0.0 -> xyz=0.07600000000000001 -0.109713 0.0470002 rpy=0.0 -0.0 0.0
- joint lleg_crotch_p_joint: origin xyz=1.15 0.0 -0.535484 rpy=0.0 -0.0 0.0 -> xyz=0.11499999999999999 0.0 -0.053548399999999996 rpy=0.0 -0.0 0.0
- joint lleg_crotch_r_mimic_joint: origin xyz=1.82901 0.0028688 0.398817 rpy=0.0 -0.0 0.0 -> xyz=0.182901 0.00028688 0.0398817 rpy=0.0 -0.0 0.0
- joint lleg_crotch_y_joint: origin xyz=-1e-07 0.0 -0.684516 rpy=0.0 -0.0 0.0 -> xyz=-1e-08 0.0 -0.0684516 rpy=0.0 -0.0 0.0
- joint lleg_knee_p2_joint: origin xyz=-3e-07 -0.162996 -0.408183 rpy=-9.99999997475e-07 -0.0 0.0 -> xyz=-3e-08 -0.0162996 -0.0408183 rpy=-9.99999997475e-07 -0.0 0.0
- joint lleg_knee_p_joint: origin xyz=0.0 0.423796 -2.71182 rpy=0.0 -0.0 0.0 -> xyz=0.0 0.0423796 -0.271182 rpy=0.0 -0.0 0.0
- joint rarm_elbow_p2_joint: origin xyz=2e-07 0.0 0.0 rpy=1.99999999495e-06 -0.0 0.0 -> xyz=2e-08 0.0 0.0 rpy=1.99999999495e-06 -0.0 0.0
- joint rarm_elbow_p_joint: origin xyz=6e-07 2.88e-05 -1.55024 rpy=-3.0000001061e-06 -9.99999997475e-07 0.0 -> xyz=6e-08 2.88e-06 -0.15502400000000002 rpy=-3.0000001061e-06 -9.99999997475e-07 0.0
- joint rarm_gripper_index0_mimic_joint: origin xyz=0.0684011 -0.310731 -0.883256 rpy=0.0 -0.0 0.0 -> xyz=0.006840110000000001 -0.0310731 -0.0883256 rpy=0.0 -0.0 0.0
- joint rarm_gripper_index1_mimic_joint: origin xyz=0.0498386 -9e-07 -0.295347 rpy=0.0 -0.0 0.0 -> xyz=0.00498386 -9e-08 -0.029534700000000004 rpy=0.0 -0.0 0.0
- joint rarm_gripper_index2_mimic_joint: origin xyz=-1.3e-06 -1e-06 -0.366376 rpy=0.0 -0.0 0.0 -> xyz=-1.3e-07 -1e-07 -0.0366376 rpy=0.0 -0.0 0.0
- joint rarm_gripper_joint: origin xyz=0.2652 -0.284142 -0.112511 rpy=0.0 -0.0 0.0 -> xyz=0.026520000000000002 -0.0284142 -0.0112511 rpy=0.0 -0.0 0.0
- joint rarm_gripper_little0_mimic_joint: origin xyz=0.0684013 0.310821 -0.812965 rpy=0.0 -0.0 0.0 -> xyz=0.00684013 0.0310821 -0.08129650000000001 rpy=0.0 -0.0 0.0
- joint rarm_gripper_little1_mimic_joint: origin xyz=0.0498386 -8e-07 -0.295347 rpy=0.0 -0.0 0.0 -> xyz=0.00498386 -8e-08 -0.029534700000000004 rpy=0.0 -0.0 0.0
- joint rarm_gripper_little2_mimic_joint: origin xyz=-1e-06 -1.1e-06 -0.366376 rpy=0.0 -0.0 0.0 -> xyz=-1e-07 -1.1e-07 -0.0366376 rpy=0.0 -0.0 0.0
- joint rarm_gripper_middle0_mimic_joint: origin xyz=0.068401 -0.105633 -0.907139 rpy=0.0 -0.0 0.0 -> xyz=0.006840100000000001 -0.010563300000000001 -0.09071390000000001 rpy=0.0 -0.0 0.0
- joint rarm_gripper_middle1_mimic_joint: origin xyz=0.0498394 -8e-07 -0.295347 rpy=0.0 -0.0 0.0 -> xyz=0.00498394 -8e-08 -0.029534700000000004 rpy=0.0 -0.0 0.0
- joint rarm_gripper_middle2_mimic_joint: origin xyz=-1.1e-06 -1.2e-06 -0.366376 rpy=0.0 -0.0 0.0 -> xyz=-1.1e-07 -1.2e-07 -0.0366376 rpy=0.0 -0.0 0.0
- joint rarm_gripper_ring0_mimic_joint: origin xyz=0.0684015 0.098905 -0.872841 rpy=0.0 -0.0 0.0 -> xyz=0.006840150000000001 0.009890500000000002 -0.0872841 rpy=0.0 -0.0 0.0
- joint rarm_gripper_ring1_mimic_joint: origin xyz=0.0498388 -9e-07 -0.295347 rpy=-9.99999997475e-07 -0.0 0.0 -> xyz=0.00498388 -9e-08 -0.029534700000000004 rpy=-9.99999997475e-07 -0.0 0.0
- joint rarm_gripper_ring2_mimic_joint: origin xyz=-1.1e-06 -1e-06 -0.366376 rpy=0.0 -0.0 0.0 -> xyz=-1.1e-07 -1e-07 -0.0366376 rpy=0.0 -0.0 0.0
- joint rarm_gripper_thumb1_mimic_joint: origin xyz=-6e-07 -0.248848 -0.170409 rpy=-1.99999999495e-06 1.99999999495e-06 0.0 -> xyz=-6e-08 -0.024884800000000002 -0.0170409 rpy=-1.99999999495e-06 1.99999999495e-06 0.0
- joint rarm_gripper_thumb2_mimic_joint: origin xyz=4e-07 -2.54e-05 -0.366319 rpy=0.0 -1.99999999495e-06 0.0 -> xyz=4e-08 -2.5400000000000002e-06 -0.0366319 rpy=0.0 -1.99999999495e-06 0.0
- joint rarm_shoulder_p_joint: origin xyz=-1.72 0.35 1.07245 rpy=0.0 -0.0 0.0 -> xyz=-0.17200000000000001 0.034999999999999996 0.107245 rpy=0.0 -0.0 0.0
- joint rarm_shoulder_r_joint: origin xyz=-0.93 -4e-07 2.29e-05 rpy=0.0 1.99999999495e-06 0.0 -> xyz=-0.09300000000000001 -4e-08 2.29e-06 rpy=0.0 1.99999999495e-06 0.0
- joint rarm_shoulder_y_joint: origin xyz=1e-06 -9e-07 -0.604907 rpy=0.0 -1.99999999495e-06 0.0 -> xyz=1e-07 -9e-08 -0.0604907 rpy=0.0 -1.99999999495e-06 0.0
- joint rarm_wrist_r_joint: origin xyz=-0.136881 -1e-07 -0.209745 rpy=1.99999999495e-06 1.99999999495e-06 0.0 -> xyz=-0.013688100000000002 -1e-08 -0.0209745 rpy=1.99999999495e-06 1.99999999495e-06 0.0
- joint rarm_wrist_y_joint: origin xyz=-1e-06 -3.74e-05 -2.51486 rpy=-9.99999997475e-07 -1.99999999495e-06 0.0 -> xyz=-1e-07 -3.74e-06 -0.25148600000000004 rpy=-9.99999997475e-07 -1.99999999495e-06 0.0
- joint rleg_ankle_p_joint: origin xyz=-0.000301 0.221804 -6.02553 rpy=0.0 9.99999997475e-07 0.0 -> xyz=-3.01e-05 0.022180400000000003 -0.602553 rpy=0.0 9.99999997475e-07 0.0
- joint rleg_ankle_p_mimic_joint: origin xyz=3e-07 1e-07 0.0 rpy=0.0 -9.99999997475e-07 0.0 -> xyz=3e-08 1e-08 0.0 rpy=0.0 -9.99999997475e-07 0.0
- joint rleg_ankle_r_joint: origin xyz=0.0011439 -1.44561 -0.716286 rpy=4.99999987365e-06 -0.0 1.5707753268 -> xyz=0.00011439000000000001 -0.14456100000000002 -0.0716286 rpy=4.99999987365e-06 -0.0 1.5707753268
- joint rleg_ankle_r_mimic_joint: origin xyz=2.99e-05 -5e-07 -0.716289 rpy=3.0000001061e-06 -0.0 1.5707763268 -> xyz=2.99e-06 -5e-08 -0.0716289 rpy=3.0000001061e-06 -0.0 1.5707763268
- joint rleg_crotch_p_back_mimic_joint: origin xyz=-0.76 1.10287 0.470002 rpy=0.0 -0.0 0.0 -> xyz=-0.07600000000000001 0.11028700000000001 0.0470002 rpy=0.0 -0.0 0.0
- joint rleg_crotch_p_front_mimic_joint: origin xyz=-0.76 -1.09713 0.469961 rpy=0.0 -0.0 0.0 -> xyz=-0.07600000000000001 -0.109713 0.046996100000000006 rpy=0.0 -0.0 0.0
- joint rleg_crotch_p_joint: origin xyz=-1.15 1e-07 -0.535484 rpy=0.0 -0.0 0.0 -> xyz=-0.11499999999999999 1e-08 -0.053548399999999996 rpy=0.0 -0.0 0.0
- joint rleg_crotch_r_mimic_joint: origin xyz=-1.82901 0.0028688 0.398817 rpy=0.0 -0.0 0.0 -> xyz=-0.182901 0.00028688 0.0398817 rpy=0.0 -0.0 0.0
- joint rleg_crotch_y_joint: origin xyz=0.0 0.0 -0.684517 rpy=0.0 -0.0 0.0 -> xyz=0.0 0.0 -0.0684517 rpy=0.0 -0.0 0.0
- joint rleg_knee_p2_joint: origin xyz=-4.01e-05 -0.162996 -0.408183 rpy=0.0 -0.0 0.0 -> xyz=-4.01e-06 -0.0162996 -0.0408183 rpy=0.0 -0.0 0.0
- joint rleg_knee_p_joint: origin xyz=1e-07 0.423796 -2.71182 rpy=0.0 -0.0 0.0 -> xyz=1e-08 0.0423796 -0.271182 rpy=0.0 -0.0 0.0
- joint rx78_Null_007_joint: origin xyz=-7e-07 4e-07 1.2322 rpy=0.0 -0.0 -0.785398163397 -> xyz=-7e-08 4e-08 0.12322 rpy=0.0 -0.0 -0.785398163397
- joint rx78_Null_008_joint: origin xyz=0.0 -3e-07 0.0 rpy=0.0 -0.0 0.0 -> xyz=0.0 -3e-08 0.0 rpy=0.0 -0.0 0.0
- joint rx78_Null_009_joint: origin xyz=1.84713 1.55851 1.94337 rpy=0.0 -0.0 -1.57079532679 -> xyz=0.18471300000000002 0.15585100000000002 0.194337 rpy=0.0 -0.0 -1.57079532679
- joint rx78_Null_010_joint: origin xyz=0.0 -1e-07 1.5e-06 rpy=0.0 -0.0 0.0 -> xyz=0.0 -1e-08 1.5000000000000002e-07 rpy=0.0 -0.0 0.0
- joint rx78_Null_011_joint: origin xyz=5e-07 -2e-07 1.2322 rpy=0.0 -0.0 0.785398163397 -> xyz=5e-08 -2e-08 0.12322 rpy=0.0 -0.0 0.785398163397
- joint rx78_Null_012_joint: origin xyz=1.84712 -1.5585 1.94337 rpy=0.0 -0.0 -1.57079532679 -> xyz=0.18471200000000002 -0.15585000000000002 0.194337 rpy=0.0 -0.0 -1.57079532679
- joint rx78_Null_042_joint: origin xyz=-1.30974 0.373955 -0.538725 rpy=3.14159265359 9.99999997475e-07 -1.57079632679 -> xyz=-0.130974 0.0373955 -0.053872500000000004 rpy=3.14159265359 9.99999997475e-07 -1.57079632679
- joint rx78_Null_043_joint: origin xyz=-1.30974 -0.374037 -0.538725 rpy=3.14159265359 9.99999997475e-07 -1.57079632679 -> xyz=-0.130974 -0.037403700000000005 -0.053872500000000004 rpy=3.14159265359 9.99999997475e-07 -1.57079632679
- joint rx78_Null_044_joint: origin xyz=0.573261 0.801901 -0.602815 rpy=0.0 9.99999997475e-07 -1.57079632679 -> xyz=0.057326100000000005 0.0801901 -0.0602815 rpy=0.0 9.99999997475e-07 -1.57079632679
- joint rx78_Null_045_joint: origin xyz=0.57326 -0.801899 -0.602816 rpy=0.0 9.99999997475e-07 -1.57079632679 -> xyz=0.057326 -0.08018990000000001 -0.060281600000000005 rpy=0.0 9.99999997475e-07 -1.57079632679
- joint rx78_Null_048_joint: origin xyz=0.28 -0.019188 0.0 rpy=0.0 -0.0 0.0 -> xyz=0.028000000000000004 -0.0019188 0.0 rpy=0.0 -0.0 0.0
- joint rx78_Null_065_joint: origin xyz=-4e-07 0.0 0.0 rpy=0.0 -0.0 0.0 -> xyz=-4e-08 0.0 0.0 rpy=0.0 -0.0 0.0
- joint rx78_Null_081_joint: origin xyz=-0.279999 -4e-07 3.05e-05 rpy=-3.0000001061e-06 -0.0 0.0 -> xyz=-0.0279999 -4e-08 3.05e-06 rpy=-3.0000001061e-06 -0.0 0.0
- joint rx78_Null_082_joint: origin xyz=-5e-07 -1.30287 -0.837529 rpy=0.0349060820064 -0.0 0.0 -> xyz=-5e-08 -0.13028700000000001 -0.0837529 rpy=0.0349060820064 -0.0 0.0
- joint rx78_Null_083_joint: origin xyz=0.0 0.0 11.5 rpy=0.0 -0.0 1.57079632679 -> xyz=0.0 0.0 1.1500000000000001 rpy=0.0 -0.0 1.57079632679
- joint rx78_Null_092_joint: origin xyz=-1.30973 0.374846 -0.538731 rpy=-3.14159165359 -3.999999989e-06 -1.5707753268 -> xyz=-0.130973 0.0374846 -0.0538731 rpy=-3.14159165359 -3.999999989e-06 -1.5707753268
- joint rx78_Null_093_joint: origin xyz=-1.30971 -0.373144 -0.538727 rpy=-3.14159165359 -3.999999989e-06 -1.5707753268 -> xyz=-0.130971 -0.0373144 -0.053872699999999996 rpy=-3.14159165359 -3.999999989e-06 -1.5707753268
- joint rx78_Null_094_joint: origin xyz=0.573261 0.802745 -0.602821 rpy=9.99999997475e-07 -3.999999989e-06 -1.5707753268 -> xyz=0.057326100000000005 0.08027450000000001 -0.060282100000000005 rpy=9.99999997475e-07 -3.999999989e-06 -1.5707753268
- joint rx78_Null_095_joint: origin xyz=0.573295 -0.801055 -0.602814 rpy=9.99999997475e-07 -3.999999989e-06 -1.5707753268 -> xyz=0.057329500000000005 -0.0801055 -0.0602814 rpy=9.99999997475e-07 -3.999999989e-06 -1.5707753268
- joint torso_lthrust_p_joint: origin xyz=2.09633 -0.644748 -0.765126 rpy=0.0 -0.0 -1.57079532679 -> xyz=0.209633 -0.0644748 -0.0765126 rpy=0.0 -0.0 -1.57079532679
- joint torso_rthrust_p_joint: origin xyz=2.09633 0.644753 -0.765126 rpy=0.0 -0.0 -1.57079532679 -> xyz=0.209633 0.0644753 -0.0765126 rpy=0.0 -0.0 -1.57079532679
- joint torso_waist_p2_joint: origin xyz=0.0 0.0028689 1.07753 rpy=0.0 -0.0 0.0 -> xyz=0.0 0.00028689000000000004 0.10775300000000002 rpy=0.0 -0.0 0.0
- joint torso_waist_p_joint: origin xyz=0.0 0.0 0.8 rpy=0.0 -0.0 0.0 -> xyz=0.0 0.0 0.08000000000000002 rpy=0.0 -0.0 0.0
- joint torso_waist_y_joint: origin xyz=1e-07 0.0 12.0 rpy=0.0 -0.0 1.57079632679 -> xyz=1e-08 0.0 1.2000000000000002 rpy=0.0 -0.0 1.57079632679
